File: board.kicad_pcb (KiCad board)
At the start: 6 copper layers, 197 x 140.5 mm, 100 parts, among them J2 Conn_2Rows-33Pins, J3 Conn_2Rows-33Pins, J4 Conn_2Rows-33Pins, J5 Conn_2Rows-33Pins, J6 Conn_2Rows-33Pins, J7 Conn_2Rows-33Pins, U1 MC68060RC50, U10 74LVC162245ADGG, U11 74LVC162245ADGG, U12 SIT2001BI-S2-33E-50.000000G, U13 74LVC162245ADGG, U2 XC95144XL-5TQG100C, U3 SST39VF1601C-70-4C-EKE, U4 IS61WV51216BLL-10TLI, U5 IS61WV51216BLL-10TLI, U6 SST39VF1601C-70-4C-EKE, U7 74LVC162245ADGG, U8 74LVC162245ADGG, U9 74LVC162245ADGG

Commit message: Added new CPLD
Parts:
- U2: value XC95144XL-5TQG100C -> XC95144XL-TQ144; footprint cpld 144:100-TQFP_XIL -> Package_QFP:TQFP-144_20x20mm_P0.5mm
- moved ? 48.1 mm to (152.1, 57.2)
- moved ? 48.1 mm to (152.1, 59.2)
- moved ? 48.1 mm to (145.1, 58.5)
- moved ? 48.1 mm to (145.1, 57.0)
- moved ? 48.1 mm to (136.5, 103.8)
- moved ? 48.1 mm to (214.0, 77.2)
- moved ? 48.1 mm to (210.0, 58.7)
- moved ? 48.1 mm to (205.9, 132.2)
- moved ? 48.1 mm to (211.4, 132.2)
- moved ? 48.1 mm to (208.4, 58.7)
- moved ? 48.1 mm to (207.5, 134.2)
- moved ? 48.1 mm to (143.5, 90.7)
- moved ? 48.1 mm to (177.4, 85.2)
- moved ? 48.1 mm to (213.0, 132.2)
- moved ? 48.1 mm to (130.5, 102.8)
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Connections:
- J6 pad 10: /EXT_CTRLOUT4 -> /EXT-SPI-CS-LATCH
- J6 pad 12: /EXT_CTRLOUT5 -> unconnected-(J6-Pin_12-Pad12)
- J6 pad 14: /EXT_CTRLOUT6 -> unconnected-(J6-Pin_14-Pad14)
- J6 pad 16: /EXT_CTRLOUT7 -> unconnected-(J6-Pin_16-Pad16)
- J6 pad 18: /EXT_CTRLOUT8 -> /EXT_CTRLOUT0
- J6 pad 2: /EXT_CTRLOUT0 -> /EXT-CLK
- J6 pad 20: /EXT_CTRLOUT9 -> /EXT_CTRLOUT1
- J6 pad 22: /EXT_CTRLOUT10 -> /EXT_CTRLOUT2
- J6 pad 24: /EXT_CTRLOUT11 -> /EXT_CTRLOUT3
- J6 pad 26: /EXT_CTRLOUT12 -> /EXT_CTRLOUT4
- J6 pad 28: /EXT_CTRLOUT13 -> /EXT_CTRLOUT5
- J6 pad 30: /EXT_CTRLOUT14 -> /EXT_CTRLOUT6
- J6 pad 32: /EXT_CTRLOUT15 -> /EXT_CTRLOUT7
- J6 pad 4: /EXT_CTRLOUT1 -> /EXT-CLKEN
- J6 pad 6: /EXT_CTRLOUT2 -> /EXT-SPI-SCLK
- J6 pad 8: /EXT_CTRLOUT3 -> /EXT-SPI-MOSI
- J7 pad 18: unconnected-(J7-Pin_18-Pad18) -> /EXT-SPI-MISO
- U1 pad M1: unconnected-(U1A-A13-PadM1) -> /A13
- U1 pad P15: unconnected-(U1C-*SNOOP-PadP15) -> /U1C-SNOOP
- U1 pad R18: unconnected-(U1C-*LOCKE-PadR18) -> /U1C-LOCKE
- U1 pad S18: unconnected-(U1C-*LOCK-PadS18) -> /U1C-LOCK
- U11 pad 11: /EXT_CTRLOUT6 -> unconnected-(U11-1B6-Pad11)
- U11 pad 12: /EXT_CTRLOUT7 -> unconnected-(U11-1B7-Pad12)
- U11 pad 13: /EXT_CTRLOUT8 -> /EXT_CTRLOUT0
- U11 pad 14: /EXT_CTRLOUT9 -> /EXT_CTRLOUT1
- U11 pad 16: /EXT_CTRLOUT10 -> /EXT_CTRLOUT2
- U11 pad 17: /EXT_CTRLOUT11 -> /EXT_CTRLOUT3
- U11 pad 19: /EXT_CTRLOUT12 -> /EXT_CTRLOUT4
- U11 pad 2: /EXT_CTRLOUT0 -> /EXT-CLK
- U11 pad 20: /EXT_CTRLOUT13 -> /EXT_CTRLOUT5
- U11 pad 22: /EXT_CTRLOUT14 -> /EXT_CTRLOUT6
- U11 pad 23: /EXT_CTRLOUT15 -> /EXT_CTRLOUT7
- U11 pad 3: /EXT_CTRLOUT1 -> /EXT-CLKEN
- U11 pad 41: unconnected-(U11-1A4-Pad41) -> /SPI-CS-LATCH
- U11 pad 43: unconnected-(U11-1A3-Pad43) -> /SPI-MOSI
- U11 pad 44: unconnected-(U11-1A2-Pad44) -> /SPI-SCLK
- U11 pad 5: /EXT_CTRLOUT2 -> /EXT-SPI-SCLK
- U11 pad 6: /EXT_CTRLOUT3 -> /EXT-SPI-MOSI
- U11 pad 8: /EXT_CTRLOUT4 -> /EXT-SPI-CS-LATCH
- U11 pad 9: /EXT_CTRLOUT5 -> unconnected-(U11-1B5-Pad9)
- U13 pad 13: unconnected-(U13-2B0-Pad13) -> /EXT-SPI-MISO
- U13 pad 36: unconnected-(U13-2A0-Pad36) -> /SPI-MISO
- U2 pad 1: /A23 -> /VCC
- U2 pad 10: /A31 -> /CPLD_X7
- U2 pad 100: /GND -> /BS2
- U2 pad 11: /CPLD_X0 -> unconnected-(U2-P11-Pad11)
- U2 pad 12: /CPLD_X1 -> unconnected-(U2-P12-Pad12)
- U2 pad 13: /CPLD_X2 -> unconnected-(U2-P13-Pad13)
- U2 pad 14: /CPLD_X3 -> unconnected-(U2-P14-Pad14)
- U2 pad 15: /CPLD_X4 -> unconnected-(U2-P15-Pad15)
- U2 pad 16: /CPLD_X5 -> /CPLD_XIN0
- U2 pad 17: /CPLD_X6 -> /CPLD_XIN1
- U2 pad 18: /CPLD_X7 -> /GND
- U2 pad 19: /CPLD_XIN0 -> /CPLD_XIN2
- U2 pad 2: /A24 -> /CPLD_X0
- U2 pad 20: /CPLD_XIN1 -> /CPLD_XIN3
- U2 pad 21: /GND -> /CPLD_XIN4
- U2 pad 22: /U1B-CLK -> /CPLD_XIN5
- U2 pad 23: /CPLD_XIN2 -> /CPLD_XIN6
- U2 pad 24: /CPLD_XIN3 -> /CPLD_XIN7
- U2 pad 25: /CPLD_XIN4 -> /SPI-MISO
- U2 pad 26: /VCC -> unconnected-(U2-P26-Pad26)
- U2 pad 27: /CPLD_XIN5 -> unconnected-(U2-P27-Pad27)
- U2 pad 28: /CPLD_XIN6 -> unconnected-(U2-P28-Pad28)
- U2 pad 29: /CPLD_XIN7 -> /GND
- U2 pad 3: /A25 -> /CPLD_X1
- U2 pad 30: unconnected-(U2-IO-Pad30) -> /U1B-CLK
- U2 pad 31: /GND -> unconnected-(U2-P31-Pad31)
- U2 pad 36: unconnected-(U2-IO-Pad36) -> /GND
- U2 pad 37: /RW -> /VCC
- U2 pad 38: /VCC -> /EPROM_OE
- U2 pad 39: /RAM_CS -> /EPROM_CS
- U2 pad 4: /A26 -> /CPLD_X2
- U2 pad 40: /RAM_OE -> /RAM_CS
- U2 pad 41: /EPROM_CS -> /RAM_OE
- U2 pad 42: /EPROM_OE -> /VCC
- U2 pad 43: /U1C-TM1 -> /RW
- U2 pad 44: /GND -> unconnected-(U2-P44-Pad44)
- U2 pad 45: /U1C-TM0 -> unconnected-(U2-P45-Pad45)
- U2 pad 46: /U1C-BR -> unconnected-(U2-P46-Pad46)
- U2 pad 47: /U1C-TM2 -> /GND
- U2 pad 48: /U1C-BB -> unconnected-(U2-P48-Pad48)
- U2 pad 49: /U1C-CLA -> unconnected-(U2-P49-Pad49)
- U2 pad 5: /VCC -> /CPLD_X3
- U2 pad 50: /U1C-TS -> /A8
- U2 pad 51: /VCC -> /A9
- U2 pad 52: /U1C-PST3 -> unconnected-(U2-P52-Pad52)
- U2 pad 53: /U1C-RW -> unconnected-(U2-P53-Pad53)
- U2 pad 54: /U1C-PST0 -> unconnected-(U2-P54-Pad54)
- U2 pad 55: /U1C-TIP -> /VCC
- U2 pad 56: /U1C-PST1 -> /A1
- U2 pad 57: /VCC -> /A0
- U2 pad 58: /U1C-TA -> /U1C-TM1
- U2 pad 59: /U1C-BTT -> /U1C-TM0
- U2 pad 6: /A27 -> /CPLD_X4
- U2 pad 60: /U1C-BG -> /U1C-LOCK
- U2 pad 61: /U1C-PST2 -> /U1C-BR
- U2 pad 63: /U1C-SAS -> unconnected-(U2-TDI-Pad63)
- U2 pad 64: /U1C-PST4 -> /U1C-LOCKE
- U2 pad 65: /U1C-BGR -> unconnected-(U2-TMS-Pad65)
- U2 pad 66: /U1C-AVEC -> /U1C-TM2
- U2 pad 67: /U1C-TCI -> unconnected-(U2-TCK-Pad67)
- U2 pad 68: /U1B-CLK -> /U1C-BB
- U2 pad 69: /GND -> /U1C-CLA
- U2 pad 7: /A28 -> /CPLD_X5
- U2 pad 70: /U1B-IPL0 -> /U1C-TS
- U2 pad 71: /U1B-CLKEN -> /U1C-PST3
- U2 pad 72: /U1B-IPL1 -> /GND
- U2 pad 73: /U1B-RSTI -> /VCC
- U2 pad 74: /BS3 -> /U1C-RW
- U2 pad 75: /GND -> /U1C-SNOOP
- U2 pad 76: /U1B-IPL2 -> /U1C-PST0
- U2 pad 77: /U1B-MDIS -> /U1C-TIP
- U2 pad 78: /BS2 -> /U1C-PST1
- U2 pad 79: /BS1 -> /U1C-TA
- U2 pad 8: /A29 -> /VCC
- U2 pad 80: /BS0 -> /U1C-BTT
- U2 pad 81: /U1B-RSTO -> /U1C-BG
- U2 pad 82: /U1B-UPA0 -> /U1C-PST2
- U2 pad 83: /U1A-TT0 -> /U1C-SAS
- U2 pad 84: /GND -> /VCC
- U2 pad 85: /U1A-TT1 -> /U1C-PST4
- U2 pad 86: /U1B-IPEND -> /U1C-BGR
- U2 pad 87: /U1A-UPA1 -> /U1C-AVEC
- U2 pad 88: /VCC -> /U1C-TCI
- U2 pad 89: /A14 -> /GND
- U2 pad 9: /A30 -> /CPLD_X6
- U2 pad 90: /A15 -> /GND
- U2 pad 91: /A16 -> /U1B-CLK
- U2 pad 92: /A17 -> /U1B-IPL0
- U2 pad 93: /A18 -> /U1B-CLKEN
- U2 pad 94: /A19 -> /U1B-IPL1
- U2 pad 95: /A20 -> /U1B-RSTI
- U2 pad 96: /A21 -> /BS3
- U2 pad 97: /A22 -> /U1B-IPL2
- U2 pad 98: /VCC -> /U1B-MDIS
- U2 pad 99: unconnected-(U2-I/O/GSR-Pad99) -> /GND
Routing:
- net /A9: track 239.7 -> 320.0 mm
- net /A8: track 236.1 -> 315.5 mm
- net /A1: track 229.6 -> 293.1 mm
- net /A0: track 185.7 -> 245.8 mm
- net /A13: track 288.3 -> 335.7 mm
- net /A12: track 291.0 -> 334.8 mm
- net /SPI-MISO: track 0.00 -> 43.4 mm
- net /U1C-LOCK: track 0.00 -> 41.2 mm
- net /U1C-LOCKE: track 0.00 -> 41.1 mm
- net /A10: track 305.8 -> 346.5 mm
- net /A11: track 298.5 -> 336.2 mm
- net /U1C-SNOOP: track 0.00 -> 37.7 mm
- net /EXT-CLK: track 0.00 -> 33.2 mm
- net /U1C-BGR: track 0.00 -> 33.2 mm
- net /EXT-CLKEN: track 0.00 -> 31.2 mm
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Other:
- board size 197 x 140.5 mm -> 206 x 115 mm
