File: board.kicad_sch (KiCad schematic)
At the start: 19 parts, among them J2 Conn_2Rows-33Pins, J3 Conn_2Rows-33Pins, J4 Conn_2Rows-33Pins, J5 Conn_2Rows-33Pins, J6 Conn_2Rows-33Pins, J7 Conn_2Rows-33Pins, U1 MC68060RC50, U10 74LVC162245ADGG, U11 74LVC162245ADGG, U12 SIT2001BI-S2-33E-50.000000G, U13 74LVC162245ADGG, U2 XC95144XL-5TQG100C, U3 SST39VF1601C-70-4C-EKE, U4 IS61WV51216BLL-10TLI, U5 IS61WV51216BLL-10TLI, U6 SST39VF1601C-70-4C-EKE, U7 74LVC162245ADGG, U8 74LVC162245ADGG, U9 74LVC162245ADGG

Commit message: Added new CPLD
Parts:
- U2: value XC95144XL-5TQG100C -> XC95144XL-TQ144; footprint 100-TQFP_XIL -> Package_QFP:TQFP-144_20x20mm_P0.5mm; symbol CPLD 144:XC95144XL-5TQG100C -> CPLD_Xilinx:XC95144XL-TQ144
Connections:
- net EXT_CTRLOUT10 is gone; now on net EXT_CTRLOUT2: J6.22 (Pin_22), U11.16 (2B2)
- net EXT_CTRLOUT11 is gone; now on net EXT_CTRLOUT3: J6.24 (Pin_24), U11.17 (2B3)
- net EXT_CTRLOUT12 is gone; now on net EXT_CTRLOUT4: J6.26 (Pin_26), U11.19 (2B4)
- net EXT_CTRLOUT13 is gone; now on net EXT_CTRLOUT5: J6.28 (Pin_28), U11.20 (2B5)
- net EXT_CTRLOUT14 is gone; now on net EXT_CTRLOUT6: J6.30 (Pin_30), U11.22 (2B6)
- net EXT_CTRLOUT15 is gone; now on net EXT_CTRLOUT7: J6.32 (Pin_32), U11.23 (2B7)
- net EXT_CTRLOUT8 is gone; now on net EXT_CTRLOUT0: J6.18 (Pin_18), U11.13 (2B0)
- net EXT_CTRLOUT9 is gone; now on net EXT_CTRLOUT1: J6.20 (Pin_20), U11.14 (2B1)
- net A0: now also U2.57 (P57)
- net A1: now also U2.56 (P56)
- net A10: now also U2.112 (P112)
- net A11: now also U2.105 (P105)
- net A12: now also U2.113 (P113)
- net A13: now also U1.M1 (A13), U2.115 (P115)
- net A14: now also U2.116 (P116); no longer U2.89 (NC)
- net A15: now also U2.117 (P117); no longer U2.90 (NC)
- net A16: now also U2.118 (P118); no longer U2.91 (NC)
- net A17: now also U2.119 (P119); no longer U2.92 (NC)
- net A18: now also U2.120 (P120); no longer U2.93 (NC)
- net A19: now also U2.121 (P121); no longer U2.94 (IO)
- net A20: now also U2.124 (P124); no longer U2.95 (IO)
- net A21: now also U2.125 (P125); no longer U2.96 (IO)
- net A22: now also U2.126 (P126); no longer U2.97 (IO)
- net A23: now also U2.128 (P128); no longer U2.1 (I/O/GTS3)
- net A24: now also U2.129 (P129); no longer U2.2 (I/O/GTS4)
- net A25: now also U2.130 (P130); no longer U2.3 (I/O/GTS1)
- net A26: now also U2.131 (P131); no longer U2.4 (I/O/GTS2)
- net A27: now also U2.132 (P132); no longer U2.6 (IO)
- net A28: now also U2.133 (P133); no longer U2.7 (IO)
- net A29: now also U2.134 (P134); no longer U2.8 (IO)
- net A30: now also U2.135 (P135); no longer U2.9 (IO)
- net A31: now also U2.136 (P136); no longer U2.10 (IO)
- net A8: now also U2.50 (P50)
- net A9: now also U2.51 (P51)
- net BS0: now also U2.102 (P102); no longer U2.80 (NC)
- net BS1: now also U2.101 (P101); no longer U2.79 (NC)
- net BS2: now also U2.100 (P100); no longer U2.78 (NC)
- net BS3: now also U2.96 (P96); no longer U2.74 (NC)
- net CPLD_X0: now also U2.2 (I/O/GTS3); no longer U2.11 (IO)
- net CPLD_X1: now also U2.3 (I/O/GTS4); no longer U2.12 (IO)
- net CPLD_X2: now also U2.4 (P4); no longer U2.13 (IO)
- net CPLD_X3: now also U2.5 (I/O/GTS1); no longer U2.14 (IO)
- net CPLD_X4: now also U2.6 (I/O/GTS2); no longer U2.15 (IO)
- net CPLD_X5: now also U2.7 (P7); no longer U2.16 (IO)
- net CPLD_X6: now also U2.9 (P9); no longer U2.17 (IO)
- net CPLD_X7: now also U2.10 (P10); no longer U2.18 (IO)
- net CPLD_XIN0: now also U2.16 (P16); no longer U2.19 (IO)
- net CPLD_XIN1: now also U2.17 (P17); no longer U2.20 (IO)
- net CPLD_XIN2: now also U2.19 (P19); no longer U2.23 (I/O/GCK2)
- net CPLD_XIN3: now also U2.20 (P20); no longer U2.24 (IO)
- net CPLD_XIN4: now also U2.21 (P21); no longer U2.25 (IO)
- net CPLD_XIN5: now also U2.22 (P22); no longer U2.27 (I/O/GCK3)
- net CPLD_XIN6: now also U2.23 (P23); no longer U2.28 (IO)
- net CPLD_XIN7: now also U2.24 (P24); no longer U2.29 (IO)
- net EPROM_CS: now also U2.39 (P39); no longer U2.41 (IO)
- net EPROM_OE: now also U2.38 (I/O/GCK3); no longer U2.42 (IO)
- net EXT_CTRLOUT0: no longer J6.2 (Pin_2), U11.2 (1B0)
- net EXT_CTRLOUT1: no longer J6.4 (Pin_4), U11.3 (1B1)
- net EXT_CTRLOUT2: no longer J6.6 (Pin_6), U11.5 (1B2)
- net EXT_CTRLOUT3: no longer J6.8 (Pin_8), U11.6 (1B3)
- net EXT_CTRLOUT4: no longer J6.10 (Pin_10), U11.8 (1B4)
- net EXT_CTRLOUT5: no longer J6.12 (Pin_12), U11.9 (1B5)
- net EXT_CTRLOUT6: no longer J6.14 (Pin_14), U11.11 (1B6)
- net EXT_CTRLOUT7: no longer J6.16 (Pin_16), U11.12 (1B7)
- net GND: now also U2.108 (GND), U2.114 (GND), U2.123 (GND), U2.144 (GND), U2.18 (GND), U2.29 (GND), U2.36 (GND), U2.47 (GND), U2.72 (GND), U2.89 (GND), U2.90 (GND), U2.99 (GND); no longer U2.100 (GND), U2.21 (GND), U2.31 (GND), U2.44 (GND), U2.69 (GND), U2.75 (GND), U2.84 (GND)
- net RAM_CS: now also U2.40 (P40); no longer U2.39 (IO)
- net RAM_OE: now also U2.41 (P41); no longer U2.40 (IO)
- net RW: now also U2.43 (P43); no longer U2.37 (IO)
- net U1A-TT0: now also U2.106 (P106); no longer U2.83 (TDO)
- net U1A-TT1: now also U2.107 (P107); no longer U2.85 (NC)
- net U1A-UPA1: now also U2.111 (P111); no longer U2.87 (NC)
- net U1B-CLK: now also U2.30 (I/O/GCK1), U2.91 (P91); no longer U2.22 (I/O/GCK1), U2.68 (NC)
- net U1B-CLKEN: now also U2.93 (P93); no longer U2.71 (NC)
- net U1B-IPEND: now also U2.110 (P110); no longer U2.86 (NC)
- net U1B-IPL0: now also U2.92 (P92); no longer U2.70 (NC)
- net U1B-IPL1: now also U2.94 (P94); no longer U2.72 (NC)
- net U1B-IPL2: now also U2.97 (P97); no longer U2.76 (NC)
- net U1B-MDIS: now also U2.98 (P98); no longer U2.77 (NC)
- net U1B-RSTI: now also U2.95 (P95); no longer U2.73 (NC)
- net U1B-RSTO: now also U2.104 (P104); no longer U2.81 (NC)
- net U1B-UPA0: now also U2.103 (P103); no longer U2.82 (NC)
- net U1C-AVEC: now also U2.87 (P87); no longer U2.66 (NC)
- net U1C-BB: now also U2.68 (P68); no longer U2.48 (TCK)
- net U1C-BG: now also U2.81 (P81); no longer U2.60 (NC)
- net U1C-BGR: now also U2.86 (P86); no longer U2.65 (NC)
- net U1C-BR: now also U2.61 (P61); no longer U2.46 (IO)
- net U1C-BTT: now also U2.80 (P80); no longer U2.59 (NC)
- net U1C-CLA: now also U2.69 (P69); no longer U2.49 (IO)
- net U1C-PST0: now also U2.76 (P76); no longer U2.54 (IO)
- net U1C-PST1: now also U2.78 (P78); no longer U2.56 (IO)
- net U1C-PST2: now also U2.82 (P82); no longer U2.61 (NC)
- net U1C-PST3: now also U2.71 (P71); no longer U2.52 (IO)
- net U1C-PST4: now also U2.85 (P85); no longer U2.64 (NC)
- net U1C-RW: now also U2.74 (P74); no longer U2.53 (IO)
- net U1C-SAS: now also U2.83 (P83); no longer U2.63 (NC)
- net U1C-TA: now also U2.79 (P79); no longer U2.58 (NC)
- net U1C-TCI: now also U2.88 (P88); no longer U2.67 (NC)
- net U1C-TIP: now also U2.77 (P77); no longer U2.55 (IO)
- net U1C-TM0: now also U2.59 (P59); no longer U2.45 (TDI)
- net U1C-TM1: now also U2.58 (P58); no longer U2.43 (IO)
- net U1C-TM2: now also U2.66 (P66); no longer U2.47 (TMS)
- net U1C-TS: now also U2.70 (P70); no longer U2.50 (IO)
- net VCC: now also U2.1 (VCCIO), U2.109 (VCCIO), U2.127 (VCCIO), U2.141 (VCCINT), U2.37 (VCCIO), U2.42 (VCCINT), U2.55 (VCCIO), U2.73 (VCCIO), U2.8 (VCCINT), U2.84 (VCCINT); no longer U2.26 (VCCIO2.5V/3.3V), U2.38 (VCCIO2.5V/3.3V), U2.5 (VCCINT3.3V), U2.51 (VCCIO2.5V/3.3V), U2.57 (VCCINT3.3V), U2.88 (VCCIO2.5V/3.3V), U2.98 (VCCINT3.3V)
- net EXT-SPI-MISO: now reaches J7.18 (Pin_18)
- net EXT-SPI-MISO: now also U13.13 (2B0)
- net U1C-SNOOP: now reaches U1.P15 (*SNOOP)
- net U1C-SNOOP: now also U2.75 (P75)
- net U1C-LOCKE: now reaches U1.R18 (*LOCKE)
- net U1C-LOCKE: now also U2.64 (P64)
- net U1C-LOCK: now reaches U1.S18 (*LOCK)
- net U1C-LOCK: now also U2.60 (P60)
- net SPI-CS-LATCH: now reaches U11.41 (1A4)
- net SPI-CS-LATCH: now also U2.139 (P139)
- net SPI-MOSI: now reaches U11.43 (1A3)
- net SPI-MOSI: now also U2.138 (P138)
- net SPI-SCLK: now reaches U11.44 (1A2)
- net SPI-SCLK: now also U2.137 (P137)
- net SPI-MISO: now reaches U13.36 (2A0)
- net SPI-MISO: now also U2.25 (P25)
- new net EXT-CLK: J6.2 (Pin_2), U11.2 (1B0)
- new net EXT-CLKEN: J6.4 (Pin_4), U11.3 (1B1)
- new net EXT-SPI-CS-LATCH: J6.10 (Pin_10), U11.8 (1B4)
- new net EXT-SPI-MOSI: J6.8 (Pin_8), U11.6 (1B3)
- new net EXT-SPI-SCLK: J6.6 (Pin_6), U11.5 (1B2)

Commit message: Added UARTs and USB host
Parts:
- added C10, C12, C5, C7: 0.1uF, Capacitor_SMD:C_1206_3216Metric_Pad1.33x1.80mm_HandSolder, symbol Device:C
- added C11, C8: 100uF, Capacitor_SMD:CP_Elec_6.3x5.4, symbol Device:C_Polarized
- added C3: 22pF, Capacitor_SMD:C_1206_3216Metric_Pad1.33x1.80mm_HandSolder, symbol Device:C
- added C4: 33pF, Capacitor_SMD:C_1206_3216Metric_Pad1.33x1.80mm_HandSolder, symbol Device:C
- added C6, C9: 10uF, Capacitor_SMD:CP_Elec_4x5.4, symbol Device:C_Polarized
- added D1, D10, D11, D2, D3, D4, D5, D6, D7, D8, D9: LED, LED_SMD:LED_1206_3216Metric, symbol Device:LED
- added J1, J8, J9: Conn_01x04, Connector_PinHeader_1.00mm:PinHeader_1x04_P1.00mm_Vertical, symbol Connector_Generic:Conn_01x04
- added R10, R11, R4, R5, R6, R7, R8, R9: 270, Resistor_SMD:R_0805_2012Metric_Pad1.20x1.40mm_HandSolder, symbol Device:R
- added R12, R13, R14: 330, Resistor_SMD:R_0805_2012Metric_Pad1.20x1.40mm_HandSolder, symbol Device:R
- added R3: 1k, Resistor_SMD:R_0805_2012Metric_Pad1.20x1.40mm_HandSolder, symbol Device:R
- added U14: SC16IS762IPW, Package_SO:TSSOP-28_4.4x9.7mm_P0.65mm, symbol Interface_UART:SC16IS762IPW
- added U15: CH9350, Package_QFP:LQFP-48_7x7mm_P0.5mm, symbol Bespoke interface chips:CH9350
- added U16, U17: AP2161W, Package_TO_SOT_SMD:SOT-23-5, symbol Power_Management:AP2161W
- added Y1: 1.8432 MHz, Crystal:Crystal_HC49-U_Vertical, symbol Device:Crystal
Connections:
- net A2: now also U2.54 (P54)
- net A3: now also U2.53 (P53)
- net A4: now also U2.52 (P52)
- net A5: now also U2.51 (P51)
- net A6: now also U2.50 (P50)
- net A7: now also U2.49 (P49)
- net A8: now also U2.46 (P46); no longer U2.50 (P50)
- net A9: now also U2.48 (P48); no longer U2.51 (P51)
- net EXT-SPI-MOSI: now also U11.5 (1B2); no longer U11.6 (1B3)
- net EXT-SPI-SCLK: now also U11.6 (1B3); no longer U11.5 (1B2)
- net GND: now also C10.2, C11.2, C12.2, C3.2, C4.2, C5.2, C6.2, C7.2, C8.2, C9.2, J1.4 (Pin_4), J8.4 (Pin_4), R12.1, R13.1, R14.2, U14.14 (SDA/VSS), U14.22 (VSS), U14.9 (I2C/~{SPI}), U15.18 (GND), U15.3 (RST), U15.4 (S0), U16.2 (GND), U16.4 (~{EN}), U17.2 (GND), U17.4 (~{EN})
- net SPI-CS-LATCH: now also U2.140 (P140); no longer U2.139 (P139)
- net SPI-MISO: now also U14.12 (n.c./SO)
- net SPI-MOSI: now also U11.44 (1A2), U14.11 (A1/SI); no longer U11.43 (1A3)
- net SPI-SCLK: now also U11.43 (1A3), U2.139 (P139), U14.13 (SCL/SCLK); no longer U11.44 (1A2), U2.137 (P137)
- net VCC: now also U10.1 (1DIR), U10.24 (2DIR), U9.1 (1DIR), U9.24 (2DIR), R10.2, R11.2, R3.1, R4.2, R5.2, R6.2, R7.2, R8.2, R9.2, U14.5 (~{RESET}), U14.8 (VDD), U15.41 (VIN5), U15.42 (VDD33)
- net UART_CS: now reaches U2.33 (P33)
- net UART_CS: now also U14.10 (A0/~{CS})
- net UART_IRQ: now reaches U2.34 (P34)
- net UART_IRQ: now also R3.2, U14.15 (~{IRQ})
- net EXT_D_DIR: now reaches U2.44 (P44)
- net EXT_D_DIR: now also U7.1 (1DIR), U7.24 (2DIR), U8.1 (1DIR), U8.24 (2DIR)
- net EXT_ADDR_OE: now reaches U2.45 (P45)
- net EXT_ADDR_OE: now also U10.25 (2OE*), U10.48 (1OE*), U9.25 (2OE*), U9.48 (1OE*)
- net EXT_D_OE: now reaches U8.25 (2OE*)
- net EXT_D_OE: now also U2.137 (P137), U7.25 (2OE*), U7.48 (1OE*), U8.48 (1OE*)
- new net: D11.1 (K), R14.1
- new net: D11.2 (A), U15.48 (LED0)
- new net: D6.1 (K), U14.20 (GPIO2/~{CDB})
- new net: D6.2 (A), R9.1
- new net: D7.1 (K), U14.19 (GPIO1/~{DTRB})
- new net: D7.2 (A), R10.1
- new net: D2.1 (K), U14.27 (GPIO6/~{CDA})
- new net: D2.2 (A), R5.1
- new net: D3.2 (A), R6.1
- new net: D5.2 (A), R8.1
- new net: D4.1 (K), U14.25 (GPIO4/~{DSRA})
- new net: D4.2 (A), R7.1
- new net: D9.1 (K), R12.2
- new net: D9.2 (A), U15.1 (LED1)
- new net: C11.1, C12.1, J8.1 (Pin_1), U17.1 (OUT)
- new net: D10.1 (K), R13.2
- new net: D8.2 (A), R11.1
- new net: D1.2 (A), R4.1
- new net: D1.1 (K), U14.28 (GPIO7/~{RIA})
- new net: J8.2 (Pin_2), U15.32 (DM)
- new net: J8.3 (Pin_3), U15.31 (DP)
- new net: C7.1, C8.1, J1.1 (Pin_1), U16.1 (OUT)
- new net: J1.2 (Pin_2), U15.30 (HM)
- new net: J1.3 (Pin_3), U15.29 (HP)
- new net: D10.2 (A), U15.2 (LED2)
- new net: D3.1 (K), U14.26 (GPIO5/~{DTRA})
- new net: J9.1 (Pin_1), U14.16 (~{CTSB})
- new net: J9.2 (Pin_2), U14.17 (~{RTSB})
- new net: D8.1 (K), U14.18 (GPIO0/~{DSRB})
- new net: D5.1 (K), U14.21 (GPIO3/~{RIB})
- new net: J9.3 (Pin_3), U14.23 (TXB)
- new net: J9.4 (Pin_4), U14.24 (RXB)
- new net: U14.3 (TXA), U15.27 (RXD)
- new net: U14.4 (RXA), U15.28 (TXD)
- new net: C3.1, U14.6 (XTAL1), Y1.2
- new net: C4.1, U14.7 (XTAL2), Y1.1
- new net VCC5: C10.1, C5.1, C6.1, C9.1, U16.5 (IN), U17.5 (IN)

Commit message: Just before changing Net names
Parts:
- added C1, C13, C14, C15, C16, C17, C18, C19, C2, C20, C21, C22, C23, C24, C25, C26, C27, C28, C29, C30, C31, C32, C33, C34, C35, C36, C37, C38, C39, C40, C41, C42, C43, C44, C45, C46, C47, C48, C49, C50, C51, C52, C53, C54, C55, C56, C57, C58, C59, C60, C61, C62: 100nF, Capacitor_SMD:C_0603_1608Metric, symbol Device:C
Connections:
- net GND: now also U13.24 (2DIR), C1.2, C13.2, C14.2, C15.2, C16.2, C17.2, C18.2, C19.2, C2.2, C20.2, C21.2, C22.2, C23.2, C24.2, C25.2, C26.2, C27.2, C28.2, C29.2, C30.2, C31.2, C32.2, C33.2, C34.2, C35.2, C36.2, C37.2, C38.2, C39.2, C40.2, C41.2, C42.2, C43.2, C44.2, C45.2, C46.2, C47.2, C48.2, C49.2, C50.2, C51.2, C52.2, C53.2, C54.2, C55.2, C56.2, C57.2, C58.2, C59.2, C60.2, C61.2, C62.2
- net UART_CS: now also U2.34 (P34); no longer U2.33 (P33)
- net UART_IRQ: now also U2.35 (P35); no longer U2.34 (P34)
- net VCC: now also U11.1 (1DIR), C1.1, C13.1, C14.1, C15.1, C16.1, C17.1, C18.1, C19.1, C2.1, C20.1, C21.1, C22.1, C23.1, C24.1, C25.1, C26.1, C27.1, C28.1, C29.1, C30.1, C31.1, C32.1, C33.1, C34.1, C35.1, C36.1, C37.1, C38.1, C39.1, C40.1, C41.1, C42.1, C43.1, C44.1, C45.1, C46.1, C47.1, C48.1, C49.1, C50.1, C51.1, C52.1, C53.1, C54.1, C55.1, C56.1, C57.1, C58.1, C59.1, C60.1, C61.1, C62.1
- net EXT_CTRLIN8: now reaches J7.20 (Pin_20)
- net EXT_CTRLIN8: now also U13.14 (2B1)
- net EXT_CTRLIN9: now reaches J7.22 (Pin_22)
- net EXT_CTRLIN9: now also U13.16 (2B2)
- net EXT_CTRLIN10: now reaches J7.24 (Pin_24)
- net EXT_CTRLIN10: now also U13.17 (2B3)
- net EXT_CTRLIN11: now reaches J7.26 (Pin_26)
- net EXT_CTRLIN11: now also U13.19 (2B4)
- net EXT_CTRLIN12: now reaches J7.28 (Pin_28)
- net EXT_CTRLIN12: now also U13.20 (2B5)
- net EXT_CTRLOUT_2OE: now reaches U2.11 (P11)
- net EXT_CTRLOUT_2OE: now also U11.25 (2OE*)
- net EXT_CTRLOUT_1OE: now reaches U2.12 (P12)
- net EXT_CTRLOUT_1OE: now also U11.48 (1OE*)
- net EXT_CTRL_2DIR: now reaches U2.13 (P13)
- net EXT_CTRL_2DIR: now also U11.24 (2DIR)
- net EXT_CTRLIN_1DIR: now reaches U2.14 (P14)
- net EXT_CTRLIN_1DIR: now also U13.1 (1DIR)
- net CPLD_X8: now reaches U2.142 (P142)
- net CPLD_X8: now also U11.40 (1A5)
- net CPLD_X9: now reaches U2.143 (I/O/GSR)
- net CPLD_X9: now also U11.38 (1A6)
- net EXT_CTRLIN_1OE: now reaches U2.15 (P15)
- net EXT_CTRLIN_1OE: now also U13.48 (1OE*)
- net CPLD_XIN8: now reaches U2.26 (P26)
- net CPLD_XIN8: now also U13.35 (2A1)
- net CPLD_XIN9: now reaches U2.27 (P27)
- net CPLD_XIN9: now also U13.33 (2A2)
- net CPLD_XIN10: now reaches U2.28 (P28)
- net CPLD_XIN10: now also U13.32 (2A3)
- net CPLD_XIN11: now reaches U2.31 (P31)
- net CPLD_XIN11: now also U13.30 (2A4)
- net CPLD_XIN12: now reaches U2.32 (I/O/GCK2)
- net CPLD_XIN12: now also U13.29 (2A5)
- net EXT_CTRLOUT9: now reaches U11.11 (1B6)
- net EXT_CTRLOUT8: now reaches U11.9 (1B5)
- net EXT_CTRLIN_2OE: now reaches U13.25 (2OE*)
- net EXT_CTRLIN_2OE: now also U2.33 (P33)
Other:
- note added: "PORT_A_OUT"
- note added: "PORT_B_BI"
- note added: "PORT_C_BI"
- note added: "PORT_D_IN"

Commit message: Now with CPLD JTAG header
Parts:
- added J10: 878311420, jtag vert conn:CONN14_878311420_MOL, symbol jtag vert conn:878311420
Connections:
- net EXT_CTRLOUT8 is gone; now on net EXT_PA0: U11.9 (1B5)
- net EXT_CTRLOUT9 is gone; now on net EXT_PA1: U11.11 (1B6)
- net EXT_D_OE is gone; now on net PD-OE: U2.137 (P137), U7.25 (2OE*), U7.48 (1OE*), U8.25 (2OE*), U8.48 (1OE*)
- net GND: now also J10.11, J10.3, J10.5, J10.7, J10.9
- net VCC: now also J10.2
- net at U2.122 (TDO): now also J10.8
- net at U2.63 (TDI): now also J10.10
- net at U2.65 (TMS): now also J10.4
- net at U2.67 (TCK): now also J10.6
- net EXT_PA0: now reaches J6.12 (Pin_12)
- net EXT_PA1: now reaches J6.14 (Pin_14)
- net CPLD_X0 renamed PB0
- net CPLD_X1 renamed PB1
- net CPLD_X2 renamed PB2
- net CPLD_X3 renamed PB3
- net CPLD_X4 renamed PB4
- net CPLD_X5 renamed PB5
- net CPLD_X6 renamed PB6
- net CPLD_X7 renamed PB7
- net CPLD_X8 renamed PA0
- net CPLD_X9 renamed PA1
- net CPLD_XIN0 renamed PC0
- net CPLD_XIN1 renamed PC1
- net CPLD_XIN10 renamed PD2
- net CPLD_XIN11 renamed PD3
- net CPLD_XIN12 renamed PD4
- net CPLD_XIN2 renamed PC2
- net CPLD_XIN3 renamed PC3
- net CPLD_XIN4 renamed PC4
- net CPLD_XIN5 renamed PC5
- net CPLD_XIN6 renamed PC6
- net CPLD_XIN7 renamed PC7
- net CPLD_XIN8 renamed PD0
- net CPLD_XIN9 renamed PD1
- net EXT-CLK renamed EXT_PA-CLK
- net EXT-CLKEN renamed EXT_PA-CLKEN
- net EXT-SPI-CS-LATCH renamed EXT_PA-SPI-CS-LATCH
- net EXT-SPI-MISO renamed EXT_PD-SPI-MISO
- net EXT-SPI-MOSI renamed EXT_PA-SPI-MOSI
- net EXT-SPI-SCLK renamed EXT_PA-SPI-SCLK
- net EXT_ADDR_OE renamed PADDR-OE
- net EXT_CTRLIN0 renamed EXT_PC0
- net EXT_CTRLIN1 renamed EXT_PC1
- net EXT_CTRLIN10 renamed EXT_PD2
- net EXT_CTRLIN11 renamed EXT_PD3
- net EXT_CTRLIN12 renamed EXT_PD4
- net EXT_CTRLIN2 renamed EXT_PC2
- net EXT_CTRLIN3 renamed EXT_PC3
- net EXT_CTRLIN4 renamed EXT_PC4
- net EXT_CTRLIN5 renamed EXT_PC5
- net EXT_CTRLIN6 renamed EXT_PC6
- net EXT_CTRLIN7 renamed EXT_PC7
- net EXT_CTRLIN8 renamed EXT_PD0
- net EXT_CTRLIN9 renamed EXT_PD1
- net EXT_CTRLIN_1DIR renamed PC-DIR
- net EXT_CTRLIN_1OE renamed PC-OE
- net EXT_CTRLIN_2OE renamed PD-OE
- net EXT_CTRLOUT0 renamed EXT_PB0
- net EXT_CTRLOUT1 renamed EXT_PB1
- net EXT_CTRLOUT2 renamed EXT_PB2
- net EXT_CTRLOUT3 renamed EXT_PB3
- net EXT_CTRLOUT4 renamed EXT_PB4
- net EXT_CTRLOUT5 renamed EXT_PB5
- net EXT_CTRLOUT6 renamed EXT_PB6
- net EXT_CTRLOUT7 renamed EXT_PB7
- net EXT_CTRLOUT_1OE renamed PA_OE
- net EXT_CTRLOUT_2OE renamed PB_OE
- net EXT_CTRL_2DIR renamed PB-DIR
- net EXT_D_DIR renamed PD-DIR

Commit message: Moved clock and added pull up/downs to TCI
Parts:
- removed C40: 100nF, Capacitor_SMD:C_0603_1608Metric, symbol Device:C
- added R15, R16, R2: 0R, Resistor_SMD:R_0805_2012Metric_Pad1.20x1.40mm_HandSolder, symbol Device:R
- U1: footprint PGA206_SOT555-4_NXP -> 68060:PGA206_SOT555-4_NXP
- U10, U11, U13, U7, U8, U9: footprint SOT362-1_NEX -> 74 buffer:SOT362-1_NEX
- U12: footprint SOT_SiT1630-S_SIT -> Clock:SOT_SiT1630-S_SIT
- U3, U6: footprint TSOP48_EKE_SST_MCH -> flash:TSOP48_EKE_SST_MCH
- U4, U5: footprint TSOP-2_44L_400MIL_ISI -> sram:TSOP-2_44L_400MIL_ISI
Connections:
- net EXT_PA-SPI-MOSI: now also U11.6 (1B3); no longer U11.5 (1B2)
- net EXT_PA-SPI-SCLK: now also U11.5 (1B2); no longer U11.6 (1B3)
- net GND: now also R15.2, R2.2
- net PD-OE: no longer U2.137 (P137), U7.25 (2OE*), U7.48 (1OE*), U8.25 (2OE*), U8.48 (1OE*)
- net U1B-CLK: now also R16.1; no longer U12.5 (OUT)
- net U1C-TBI: now also U2.88 (P88)
- net U1C-TCI: now also R15.1; no longer U2.88 (P88)
- net VUSB2: now reaches C11.1, C12.1, J8.1 (Pin_1), U17.1 (OUT)
- net USB-DM: now reaches J8.2 (Pin_2), U15.32 (DM)
- net USB-DP: now reaches J8.3 (Pin_3), U15.31 (DP)
- net VUSB1: now reaches C7.1, C8.1, J1.1 (Pin_1), U16.1 (OUT)
- net USB-HM: now reaches J1.2 (Pin_2), U15.30 (HM)
- net USB-HB: now reaches J1.3 (Pin_3), U15.29 (HP)
- net at U1.T5 (*CDIS): now also R2.1
- net UART2-CTSB: now reaches J9.1 (Pin_1), U14.16 (~{CTSB})
- net UART2-RTSB: now reaches J9.2 (Pin_2), U14.17 (~{RTSB})
- net UART2-TXB: now reaches J9.3 (Pin_3), U14.23 (TXB)
- net UART2-RXB: now reaches J9.4 (Pin_4), U14.24 (RXB)
- net PD-DIR renamed PDATA-DIR
- new net: R16.2, U12.5 (OUT)
- new net PDATA-OE: U2.137 (P137), U7.25 (2OE*), U7.48 (1OE*), U8.25 (2OE*), U8.48 (1OE*)

Commit message: X02 now all connected
Parts:
- removed U2: XC95144XL-TQ144, Package_QFP:TQFP-144_20x20mm_P0.5mm, symbol CPLD_Xilinx:XC95144XL-TQ144
- added U2: LCMXO2-7000HC-6TG144I, lattice_x02:TQFP144_LAT, symbol lattice_x02:LCMXO2-7000HC-6TG144I
Connections:
- net A0: now also U2.60 (PB29B)
- net A1: now also U2.59 (PB29A)
- net A10: now also U2.107 (PR2A)
- net A11: now also U2.100 (PR5A)
- net A12: now also U2.109 (PT36D)
- net A13: now also U2.110 (PT36C)
- net A14: now also U2.111 (PT35B)
- net A15: now also U2.112 (PT35A)
- net A16: now also U2.113 (PT33B)
- net A17: now also U2.114 (PT33A)
- net A18: now also U2.115 (PT28B)
- net A19: now also U2.117 (PT28A)
- net A2: now also U2.58 (PB26B)
- net A20: now also U2.119 (PT27D)
- net A21: now also U2.120 (PT27C)
- net A22: now also U2.121 (PT25B)
- net A23: now also U2.122 (PT25A)
- net A24: now also U2.127 (PT18B)
- net A25: now also U2.128 (PT18A)
- net A26: now also U2.132 (PT15B)
- net A27: now also U2.133 (PT15A)
- net A28: now also U2.138 (PT11B)
- net A29: now also U2.139 (PT11A)
- net A3: now also U2.57 (PB26A)
- net A30: now also U2.140 (PT10B)
- net A31: now also U2.141 (PT10A)
- net A4: now also U2.56 (PB23B)
- net A5: now also U2.55 (PB23A)
- net A6: now also U2.54 (PB18B)
- net A7: now also U2.52 (PB18A)
- net A8: now also U2.49 (PB16A)
- net A9: now also U2.50 (PB16B)
- net EPROM_CS: now also U2.35 (PL25B)
- net EPROM_OE: now also U2.34 (PL25A)
- net GND: now also U2.101 (GND), U2.116 (GND), U2.124 (GND), U2.134 (GND), U2.18 (GND), U2.29 (GND), U2.46 (GND), U2.53 (GND), U2.64 (GND), U2.8 (GND), U2.80 (GND), U2.90 (GND)
- net PADDR-OE: now also U2.42 (PB9A)
- net PA_OE: now also U2.143 (PT9A)
- net PB-DIR: now also U2.12 (PL9B)
- net PB0: now also U2.1 (PL3A)
- net PB1: now also U2.2 (PL3B)
- net PB2: now also U2.3 (PL4A)
- net PB3: now also U2.4 (PL4B)
- net PB4: now also U2.5 (PL6A)
- net PB5: now also U2.6 (PL6B)
- net PB6: now also U2.9 (PL8A)
- net PB7: now also U2.10 (PL8B)
- net PB_OE: now also U2.11 (PL9A)
- net PC-DIR: now also U2.13 (PL10A)
- net PC-OE: now also U2.14 (PL10B)
- net PC0: now also U2.15 (PL11A)
- net PC1: now also U2.17 (PL11B)
- net PC2: now also U2.19 (PL12A)
- net PC3: now also U2.20 (PL12B)
- net PC4: now also U2.21 (PL15A)
- net PC5: now also U2.22 (PL15B)
- net PC6: now also U2.23 (PL17A)
- net PC7: now also U2.24 (PL17B)
- net PD-OE: now also U2.33 (PL24B)
- net PD0: now also U2.25 (PL19A)
- net PD1: now also U2.26 (PL19B)
- net PD2: now also U2.27 (PL22A)
- net PD3: now also U2.28 (PL22B)
- net PD4: now also U2.31 (PL23D)
- net PDATA-DIR: now also U2.48 (PB13B)
- net PDATA-OE: now also U2.142 (PT9B)
- net RAM_CS: now also U2.38 (PB4A)
- net RAM_OE: now also U2.39 (PB4B)
- net RW: now also U2.41 (PB6B)
- net SPI-CS-LATCH: now also U2.40 (PB6A)
- net SPI-MISO: now also U2.45 (PB12B)
- net SPI-MOSI: now also U2.71 (PB38B)
- net SPI-SCLK: now also U2.44 (PB12A)
- net U1A-TT0: now also U2.103 (PR4C)
- net U1A-TT1: now also U2.104 (PR3B)
- net U1A-UPA1: now also U2.106 (PR2B)
- net U1B-CLK: now also U2.92 (PR12A)
- net U1B-CLKEN: now also U2.94 (PR11A)
- net U1B-IPEND: now also U2.105 (PR3A)
- net U1B-IPL0: now also U2.93 (PR11B)
- net U1B-IPL1: now also U2.95 (PR9B)
- net U1B-IPL2: now also U2.97 (PR7B)
- net U1B-RSTI: now also U2.96 (PR9A)
- net U1B-RSTO: now also U2.99 (PR5B)
- net U1B-UPA0: now also U2.98 (PR7A)
- net U1C-AVEC: now also U2.87 (PR15B)
- net U1C-BG: now also U2.82 (PR18A)
- net U1C-BGR: now also U2.86 (PR16A)
- net U1C-BR: now also U2.68 (PB37A)
- net U1C-BTT: now also U2.81 (PR18B)
- net U1C-CLA: now also U2.69 (PB37B)
- net U1C-LOCK: now also U2.67 (PB35B)
- net U1C-LOCKE: now also U2.65 (PB35A)
- net U1C-RW: now also U2.75 (PR23B)
- net U1C-SAS: now also U2.84 (PR17A)
- net U1C-SIZ0: now also U2.70 (PB38A)
- net U1C-SIZ1: now also U2.73 (PR24B)
- net U1C-SNOOP: now also U2.76 (PR23A)
- net U1C-TA: now also U2.78 (PR21A)
- net U1C-TBI: now also U2.89 (PR15A)
- net U1C-TCI: now also U2.91 (PR12B)
- net U1C-TEA: now also U2.83 (PR17B)
- net U1C-TIP: now also U2.77 (PR21B)
- net U1C-TM0: now also U2.62 (PB31B)
- net U1C-TM1: now also U2.61 (PB31A)
- net U1C-TM2: now also U2.63 (PB31D)
- net U1C-TRA: now also U2.85 (PR16B)
- net U1C-TS: now also U2.74 (PR24A)
- net UART_CS: now also U2.47 (PB13A)
- net UART_IRQ: now also U2.43 (PB9B)
- net VCC: now also U2.102 (VCCIO1), U2.108 (VCC), U2.118 (VCCIO0), U2.123 (VCCIO0), U2.135 (VCCIO0), U2.144 (VCC), U2.16 (VCCIO4), U2.30 (VCCIO3), U2.36 (VCC), U2.37 (VCCIO2), U2.51 (VCCIO2), U2.66 (VCCIO2), U2.7 (VCCIO5), U2.72 (VCC), U2.79 (VCCIO1), U2.88 (VCCIO1)
- net EXT_PD5: now reaches J7.30 (Pin_30)
- net EXT_PD5: now also U13.22 (2B6)
- net CPLD-TDO: now reaches J10.8
- net CPLD-TDO: now also U2.137 (PT14C)
- net CPLD-TDI: now reaches J10.10
- net CPLD-TDI: now also U2.136 (PT14D)
- net CPLD-TMS: now reaches J10.4
- net CPLD-TMS: now also U2.130 (PT17D)
- net CPLD-TCK: now reaches J10.6
- net CPLD-TCK: now also U2.131 (PT17C)
- net PD5: now reaches U13.27 (2A6)
- net PD5: now also U2.32 (PL24A)
- new net I2C-MCLK: U2.126 (PT22C)
- new net I2C-MDATA: U2.125 (PT22D)
Other:
- moved on the sheet: C10, C11, C12, C3, C4, C5, C53, C54, C55, C56, C57, C58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
