File: board.kicad_sch (KiCad schematic)
At the start: 120 parts, among them J1 Conn_01x04, J10 878311420, J11 Conn_01x02, J2 Conn_2Rows-33Pins, J3 Conn_2Rows-33Pins, J4 Conn_2Rows-33Pins, J5 Conn_2Rows-33Pins, J6 Conn_2Rows-33Pins, J7 Conn_2Rows-33Pins, J8 Conn_01x04, J9 Conn_01x04, U1 MC68060RC50, U10 74LVC162245ADGG, U11 74LVC162245ADGG, U12 SIT2001BI-S2-33E-50.000000G, U13 74LVC162245ADGG, U14 SC16IS762IPW, U15 CH9350, U16 AP2161W, U17 AP2161W, U18 TPS3808DBV, U19 PCA9515AD, U2 LCMXO2-7000HC-6TG144I, U3 SST39VF1601C-70-4C-EKE, U4 IS61WV204816BLL-10TLI, U5 IS61WV204816BLL-10TLI, U6 SST39VF1601C-70-4C-EKE, U7 74LVC162245ADGG, U8 74LVC162245ADGG, U9 74LVC162245ADGG, Y1 1.8432 MHz

Commit message: Re-wired to include new Everspin Flash
Parts:
- removed C48, C49, C50, C51, C52, C53, C54, C55, C56, C57, C58, C59, C60, C61, C62: 100nF, Capacitor_SMD:C_0603_1608Metric, symbol Device:C
- removed U3, U6: SST39VF1601C-70-4C-EKE, TSOP48_EKE_SST_MCH, symbol Flash:SST39VF1601C-70-4C-EKE
- added U20, U21: 74LVC162245ADGG, 74 buffer:SOT362-1_NEX, symbol 7416254 buffer:74LVC16245ADGG
- added U3, U6: MR5A16AYS35, mram:TSOP54_MR5A16_10P16X22P22_EVS, symbol mram:MR5A16AYS35
Connections:
- net A10: now also U3.23 (A8), U6.23 (A8)
- net A11: now also U3.24 (A9), U6.24 (A9)
- net A12: now also U3.31 (A10), U6.31 (A10)
- net A13: now also U3.32 (A11), U6.32 (A11)
- net A14: now also U3.33 (A12), U6.33 (A12)
- net A15: now also U3.34 (A13), U6.34 (A13)
- net A16: now also U3.35 (A14), U6.35 (A14)
- net A17: now also U3.50 (A15), U6.50 (A15)
- net A18: now also U3.51 (A16), U6.51 (A16)
- net A19: now also U3.52 (A17), U6.52 (A17)
- net A2: now also U3.3 (A0), U6.3 (A0)
- net A20: now also U3.53 (A18), U6.53 (A18)
- net A21: now also U3.2 (A19), U6.2 (A19)
- net A22: now also U3.1 (A20), U6.1 (A20)
- net A3: now also U3.4 (A1), U6.4 (A1)
- net A4: now also U3.5 (A2), U6.5 (A2)
- net A5: now also U3.6 (A3), U6.6 (A3)
- net A6: now also U3.7 (A4), U6.7 (A4)
- net A7: now also U3.20 (A5), U6.20 (A5)
- net A8: now also U3.21 (A6), U6.21 (A6)
- net A9: now also U3.22 (A7), U6.22 (A7)
- net BS0: now also U6.48 (UB)
- net BS1: now also U6.47 (LB)
- net BS2: now also U3.48 (UB)
- net BS3: now also U3.47 (LB)
- net D0: now also U20.2 (1B0)
- net D1: now also U20.3 (1B1)
- net D10: now also U20.16 (2B2)
- net D11: now also U20.17 (2B3)
- net D12: now also U20.19 (2B4)
- net D13: now also U20.20 (2B5)
- net D14: now also U20.22 (2B6)
- net D15: now also U20.23 (2B7)
- net D16: now also U21.2 (1B0)
- net D17: now also U21.3 (1B1)
- net D18: now also U21.5 (1B2)
- net D19: now also U21.6 (1B3)
- net D2: now also U20.5 (1B2)
- net D20: now also U21.8 (1B4)
- net D21: now also U21.9 (1B5)
- net D22: now also U21.11 (1B6)
- net D23: now also U21.12 (1B7)
- net D24: now also U21.13 (2B0)
- net D25: now also U21.14 (2B1)
- net D26: now also U21.16 (2B2)
- net D27: now also U21.17 (2B3)
- net D28: now also U21.19 (2B4)
- net D29: now also U21.20 (2B5)
- net D3: now also U20.6 (1B3)
- net D30: now also U21.22 (2B6)
- net D31: now also U21.23 (2B7)
- net D4: now also U20.8 (1B4)
- net D5: now also U20.9 (1B5)
- net D6: now also U20.11 (1B6)
- net D7: now also U20.12 (1B7)
- net D8: now also U20.13 (2B0)
- net D9: now also U20.14 (2B1)
- net EPROM_CS: now also U3.8 (E), U6.8 (E)
- net EPROM_OE: now also U3.49 (G), U6.49 (G)
- net GND: now also U20.10 (GND), U20.15 (GND), U20.21 (GND), U20.28 (GND), U20.34 (GND), U20.39 (GND), U20.4 (GND), U20.45 (GND), U21.10 (GND), U21.15 (GND), U21.21 (GND), U21.28 (GND), U21.34 (GND), U21.39 (GND), U21.4 (GND), U21.45 (GND), U3.14 (VSS), U3.42 (VSS), U6.14 (VSS), U6.42 (VSS)
- net RW: now also U20.1 (1DIR), U20.24 (2DIR), U21.1 (1DIR), U21.24 (2DIR), U3.19 (W), U6.19 (W)
- net VCC: now also U20.18 (VCC), U20.31 (VCC), U20.42 (VCC), U20.7 (VCC), U21.18 (VCC), U21.31 (VCC), U21.42 (VCC), U21.7 (VCC), U3.13 (VDD), U3.41 (VDD), U6.13 (VDD), U6.41 (VDD)
- net EPROM_BUFFER_OE: now reaches U2.96 (PR9A)
- net EPROM_BUFFER_OE: now also U20.25 (2OE*), U20.48 (1OE*), U21.25 (2OE*), U21.48 (1OE*)
- new net MRAM_D0: U20.47 (1A0), U3.9 (DQ0)
- new net MRAM_D1: U20.46 (1A1), U3.10 (DQ1)
- new net MRAM_D10: U20.33 (2A2), U3.44 (DQ13)
- new net MRAM_D11: U20.32 (2A3), U3.43 (DQ12)
- new net MRAM_D12: U20.30 (2A4), U3.40 (DQ11)
- new net MRAM_D13: U20.29 (2A5), U3.39 (DQ10)
- new net MRAM_D14: U20.27 (2A6), U3.38 (DQ)
- new net MRAM_D15: U20.26 (2A7), U3.37 (DQ8)
- new net MRAM_D16: U21.47 (1A0), U6.9 (DQ0)
- new net MRAM_D17: U21.46 (1A1), U6.10 (DQ1)
- new net MRAM_D18: U21.44 (1A2), U6.11 (DQ2)
- new net MRAM_D19: U21.43 (1A3), U6.12 (DQ3)
- new net MRAM_D2: U20.44 (1A2), U3.11 (DQ2)
- new net MRAM_D20: U21.41 (1A4), U6.15 (DQ4)
- new net MRAM_D21: U21.40 (1A5), U6.16 (DQ5)
- new net MRAM_D22: U21.38 (1A6), U6.17 (DQ6)
- new net MRAM_D23: U21.37 (1A7), U6.18 (DQ7)
- new net MRAM_D24: U21.36 (2A0), U6.46 (DQ15)
- new net MRAM_D25: U21.35 (2A1), U6.45 (DQ14)
- new net MRAM_D26: U21.33 (2A2), U6.44 (DQ13)
- new net MRAM_D27: U21.32 (2A3), U6.43 (DQ12)
- new net MRAM_D28: U21.30 (2A4), U6.40 (DQ11)
- new net MRAM_D29: U21.29 (2A5), U6.39 (DQ10)
- new net MRAM_D3: U20.43 (1A3), U3.12 (DQ3)
- new net MRAM_D30: U21.27 (2A6), U6.38 (DQ)
- new net MRAM_D31: U21.26 (2A7), U6.37 (DQ8)
- new net MRAM_D4: U20.41 (1A4), U3.15 (DQ4)
- new net MRAM_D5: U20.40 (1A5), U3.16 (DQ5)
- new net MRAM_D6: U20.38 (1A6), U3.17 (DQ6)
- new net MRAM_D7: U20.37 (1A7), U3.18 (DQ7)
- new net MRAM_D8: U20.36 (2A0), U3.46 (DQ15)
- new net MRAM_D9: U20.35 (2A1), U3.45 (DQ14)
Other:
- moved on the sheet: C1, C13, C14, C15, C16, C17, C18, C19, C2, C20, C21, C22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

Commit message: Added daminping resistors
Parts:
- added R18, R19, R20, R21, R22, R23, R24, R25, R26, R27, R28, R29, R30, R31, R32, R33, R34, R35, R36, R37, R38, R39, R43, R44, R45, R46, R47, R48: 33R, Resistor_SMD:R_0201_0603Metric_Pad0.64x0.40mm_HandSolder, symbol Device:R
- added R40, R41, R42: 22R, Resistor_SMD:R_0201_0603Metric_Pad0.64x0.40mm_HandSolder, symbol Device:R
- R16: value 0R -> 22R
Connections:
- net A10: now also R38.2; no longer U2.107 (PR2A), U3.23 (A8), U4.45 (A8), U5.45 (A8), U6.23 (A8), U9.33 (2A2)
- net A11: now also R37.2; no longer U2.100 (PR5A), U3.24 (A9), U4.30 (A9), U5.30 (A9), U6.24 (A9), U9.32 (2A3)
- net A12: now also R36.2; no longer U2.109 (PT36D), U3.31 (A10), U4.29 (A10), U5.29 (A10), U6.31 (A10), U9.30 (2A4)
- net A13: now also R35.2; no longer U2.110 (PT36C), U3.32 (A11), U4.28 (A11), U5.28 (A11), U6.32 (A11), U9.29 (2A5)
- net A14: now also R33.2; no longer U2.111 (PT35B), U3.33 (A12), U4.27 (A12), U5.27 (A12), U6.33 (A12), U9.27 (2A6)
- net A15: now also R31.2; no longer U2.112 (PT35A), U3.34 (A13), U4.26 (A13), U5.26 (A13), U6.34 (A13), U9.26 (2A7)
- net A16: now also R32.2; no longer U10.26 (2A7), U2.113 (PT33B), U3.35 (A14), U4.25 (A14), U5.25 (A14), U6.35 (A14)
- net A17: now also R29.2; no longer U10.27 (2A6), U2.114 (PT33A), U3.50 (A15), U4.24 (A15), U5.24 (A15), U6.50 (A15)
- net A18: now also R28.2; no longer U10.29 (2A5), U2.115 (PT28B), U3.51 (A16), U4.23 (A16), U5.23 (A16), U6.51 (A16)
- net A19: now also R30.2; no longer U10.30 (2A4), U2.117 (PT28A), U3.52 (A17), U4.22 (A17), U5.22 (A17), U6.52 (A17)
- net A2: now also R24.2; no longer U2.58 (PB26B), U3.3 (A0), U4.5 (A0), U5.5 (A0), U6.3 (A0), U9.44 (1A2)
- net A20: now also R27.2; no longer U10.32 (2A3), U2.119 (PT27D), U3.53 (A18), U4.21 (A18), U5.21 (A18), U6.53 (A18)
- net A21: now also R26.2; no longer U10.33 (2A2), U2.120 (PT27C), U3.2 (A19), U4.20 (A19), U5.20 (A19), U6.2 (A19)
- net A22: now also R34.2; no longer U10.35 (2A1), U2.121 (PT25B), U3.1 (A20), U4.31 (A20), U5.31 (A20), U6.1 (A20)
- net A3: now also R25.2; no longer U2.57 (PB26A), U3.4 (A1), U4.4 (A1), U5.4 (A1), U6.4 (A1), U9.43 (1A3)
- net A4: now also R23.2; no longer U2.56 (PB23B), U3.5 (A2), U4.3 (A2), U5.3 (A2), U6.5 (A2), U9.41 (1A4)
- net A5: now also R22.2; no longer U2.55 (PB23A), U3.6 (A3), U4.2 (A3), U5.2 (A3), U6.6 (A3), U9.40 (1A5)
- net A6: now also R20.2; no longer U2.54 (PB18B), U3.7 (A4), U4.1 (A4), U5.1 (A4), U6.7 (A4), U9.38 (1A6)
- net A7: now also R19.2; no longer U2.52 (PB18A), U3.20 (A5), U4.48 (A5), U5.48 (A5), U6.20 (A5), U9.37 (1A7)
- net A8: now also R21.1; no longer U2.49 (PB16A), U3.21 (A6), U4.47 (A6), U5.47 (A6), U6.21 (A6), U9.36 (2A0)
- net A9: now also R18.2; no longer U2.50 (PB16B), U3.22 (A7), U4.46 (A7), U5.46 (A7), U6.22 (A7), U9.35 (2A1)
- net BS0: now also R45.1; no longer U1.Q4 (*BS0)
- net BS1: now also R46.1; no longer U1.Q5 (*BS1)
- net BS2: now also R47.1; no longer U1.Q6 (*BS2)
- net BS3: now also R48.1; no longer U1.Q7 (*BS3)
- net EPROM_BUFFER_OE: now also R40.2; no longer U2.96 (PR9A)
- net EPROM_CS: now also R44.2; no longer U2.35 (PL25B)
- net EPROM_OE: now also R41.2; no longer U2.34 (PL25A)
- net RAM_CS: now also R43.1; no longer U2.38 (PB4A)
- net RAM_OE: now also R42.1; no longer U2.39 (PB4B)
- net RW: now also R39.1; no longer U2.41 (PB6B)
- new net AR10: R38.1, U2.107 (PR2A), U3.23 (A8), U4.45 (A8), U5.45 (A8), U6.23 (A8), U9.33 (2A2)
- new net AR11: R37.1, U2.100 (PR5A), U3.24 (A9), U4.30 (A9), U5.30 (A9), U6.24 (A9), U9.32 (2A3)
- new net AR12: R36.1, U2.109 (PT36D), U3.31 (A10), U4.29 (A10), U5.29 (A10), U6.31 (A10), U9.30 (2A4)
- new net AR13: R35.1, U2.110 (PT36C), U3.32 (A11), U4.28 (A11), U5.28 (A11), U6.32 (A11), U9.29 (2A5)
- new net AR14: R33.1, U2.111 (PT35B), U3.33 (A12), U4.27 (A12), U5.27 (A12), U6.33 (A12), U9.27 (2A6)
- new net AR15: R31.1, U2.112 (PT35A), U3.34 (A13), U4.26 (A13), U5.26 (A13), U6.34 (A13), U9.26 (2A7)
- new net AR16: R32.1, U10.26 (2A7), U2.113 (PT33B), U3.35 (A14), U4.25 (A14), U5.25 (A14), U6.35 (A14)
- new net AR17: R29.1, U10.27 (2A6), U2.114 (PT33A), U3.50 (A15), U4.24 (A15), U5.24 (A15), U6.50 (A15)
- new net AR18: R28.1, U10.29 (2A5), U2.115 (PT28B), U3.51 (A16), U4.23 (A16), U5.23 (A16), U6.51 (A16)
- new net AR19: R30.1, U10.30 (2A4), U2.117 (PT28A), U3.52 (A17), U4.22 (A17), U5.22 (A17), U6.52 (A17)
- new net AR2: R24.1, U2.58 (PB26B), U3.3 (A0), U4.5 (A0), U5.5 (A0), U6.3 (A0), U9.44 (1A2)
- new net AR20: R27.1, U10.32 (2A3), U2.119 (PT27D), U3.53 (A18), U4.21 (A18), U5.21 (A18), U6.53 (A18)
- new net AR21: R26.1, U10.33 (2A2), U2.120 (PT27C), U3.2 (A19), U4.20 (A19), U5.20 (A19), U6.2 (A19)
- new net AR22: R34.1, U10.35 (2A1), U2.121 (PT25B), U3.1 (A20), U4.31 (A20), U5.31 (A20), U6.1 (A20)
- new net AR3: R25.1, U2.57 (PB26A), U3.4 (A1), U4.4 (A1), U5.4 (A1), U6.4 (A1), U9.43 (1A3)
- new net AR4: R23.1, U2.56 (PB23B), U3.5 (A2), U4.3 (A2), U5.3 (A2), U6.5 (A2), U9.41 (1A4)
- new net AR5: R22.1, U2.55 (PB23A), U3.6 (A3), U4.2 (A3), U5.2 (A3), U6.6 (A3), U9.40 (1A5)
- new net AR6: R20.1, U2.54 (PB18B), U3.7 (A4), U4.1 (A4), U5.1 (A4), U6.7 (A4), U9.38 (1A6)
- new net AR7: R19.1, U2.52 (PB18A), U3.20 (A5), U4.48 (A5), U5.48 (A5), U6.20 (A5), U9.37 (1A7)
- new net AR8: R21.2, U2.50 (PB16B), U3.21 (A6), U4.47 (A6), U5.47 (A6), U6.21 (A6), U9.36 (2A0)
- new net AR9: R18.1, U2.49 (PB16A), U3.22 (A7), U4.46 (A7), U5.46 (A7), U6.22 (A7), U9.35 (2A1)
- new net BS0_INT: R45.2, U1.Q4 (*BS0)
- new net BS1_INT: R46.2, U1.Q5 (*BS1)
- new net BS2_INT: R47.2, U1.Q6 (*BS2)
- new net BS3_INT: R48.2, U1.Q7 (*BS3)
- new net EPROM_BUFFER_OE_INT: R40.1, U2.96 (PR9A)
- new net EPROM_CS_INT: R44.1, U2.35 (PL25B)
- new net EPROM_OE_INT: R41.1, U2.34 (PL25A)
- new net RAM_CS_INT: R43.2, U2.38 (PB4A)
- new net RAM_OE_INT: R42.2, U2.39 (PB4B)
- new net RW_INT: R39.2, U2.41 (PB6B)

Commit message: Resistors on Bs0-3 and A0, A1
Parts:
- added R49, R50: 33R, Resistor_SMD:R_0201_0603Metric_Pad0.64x0.40mm_HandSolder, symbol Device:R
Connections:
- net A0: now also R49.2; no longer U2.60 (PB29B), U9.47 (1A0)
- net A1: now also R50.2; no longer U2.59 (PB29A), U9.46 (1A1)
- new net AR0: R49.1, U2.60 (PB29B), U9.47 (1A0)
- new net AR1: R50.1, U2.59 (PB29A), U9.46 (1A1)
Changed lines of the file:
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@@
 	(wire
 		(pts
+			(xy 167.64 346.71) (xy 172.72 346.71)
+		)
+		(stroke
+			(width 0)
+			(type default)
+		)
+	)
+	(wire
+		(pts
 			(xy 307.34 571.5) (xy 307.34 576.58)
 		)
@@
 	(wire
 		(pts
+			(xy 167.64 336.55) (xy 172.72 336.55)
+		)
+		(stroke
+			(width 0)
+			(type default)
+		)
+	)
+	(wire
+		(pts
 			(xy 681.99 361.95) (xy 699.77 361.95)
 		)
@@
 		)
 	)
-	(label "A1"
+	(label "AR1"
 		(at 450.85 270.51 0)
 		(effects
@@
 		)
 	)
-	(label "A0"
+	(label "AR0"
 		(at 450.85 267.97 0)
 		(effects
@@
 		)
 	)
-	(label "A0"
+	(label "AR0"
 		(at 760.73 222.25 0)
 		(effects
@@
 		)
 	)
-	(label "A1"
+	(label "AR1"
 		(at 760.73 224.79 0)
 		(effects
@@
 		)
 	)
+	(label "AR0"
+		(at 167.64 346.71 0)
+		(effects
+			(font
+				(size 1.27 1.27)
+			)
+			(justify left bottom)
+		)
+	)
 	(label "GND"
 		(at 246.38 346.71 0)
@@
 		)
 	)
+	(label "AR1"
+		(at 167.64 336.55 0)
+		(effects
+			(font
+				(size 1.27 1.27)
+			)
+			(justify left bottom)
+		)
+	)
 	(label "A5"
 		(at 191.77 306.07 0)
@@
 	(symbol
 		(lib_id "Device:R")
+		(at 176.53 346.71 90)
+		(unit 1)
+		(body_style 1)
+		(exclude_from_sim no)
+		(in_bom yes)
+		(on_board yes)
+		(in_pos_files yes)
+		(dnp no)
+		(fields_autoplaced yes)
+		(property "Reference" "R49"
+			(at 176.53 340.36 90)
+			(show_name no)
+			(do_not_autoplace no)
+			(effects
+				(font
+					(size 1.27 1.27)
+				)
+			)
+		)
+		(property "Value" "33R"
+			(at 176.53 342.9 90)
+			(show_name no)
+			(do_not_autoplace no)
+			(effects
+				(font
+					(size 1.27 1.27)
+				)
+			)
+		)
+		(property "Footprint" "Resistor_SMD:R_0201_0603Metric_Pad0.64x0.40mm_HandSolder"
+			(at 176.53 348.488 90)
+			(hide yes)
+			(show_name no)
+			(do_not_autoplace no)
+			(effects
+				(font
+					(size 1.27 1.27)
+				)
+			)
+		)
+		(property "Datasheet" ""
+			(at 176.53 346.71 0)
+			(hide yes)
+			(show_name no)
+			(do_not_autoplace no)
+			(effects
+				(font
+					(size 1.27 1.27)
+				)
+			)
+		)
+		(property "Description" "Resistor"
+			(at 176.53 346.71 0)
+			(hide yes)
+			(show_name no)
+			(do_not_autoplace no)
+			(effects
+				(font
+					(size 1.27 1.27)
+				)
+			)
+		)
+		(pin "2"
+		)
+		(pin "1"
+		)
+		(instances
+			(project "board"
+				(path "/27e6fb8b-ebcf-4ece-872b-7722c171602a"
+					(reference "R49")
+					(unit 1)
+				)
+			)
+		)
+	)
+	(symbol
+		(lib_id "Device:R")
 		(at 363.22 321.31 270)
 		(mirror x)
@@
 					(unit 1)
 				)
+			)
+		)
+	)
+	(symbol
+		(lib_id "Device:R")
+		(at 176.53 336.55 90)
+		(unit 1)
+		(body_style 1)
+		(exclude_from_sim no)
+		(in_bom yes)
+		(on_board yes)
+		(in_pos_files yes)
+		(dnp no)
+		(fields_autoplaced yes)
+		(property "Reference" "R50"
+			(at 176.53 330.2 90)
+			(show_name no)
+			(do_not_autoplace no)
+			(effects
+				(font
+					(size 1.27 1.27)
+				)
+			)
+		)
+		(property "Value" "33R"
+			(at 176.53 332.74 90)
+			(show_name no)
+			(do_not_autoplace no)
+			(effects
+				(font
+					(size 1.27 1.27)
+				)
+			)
+		)
+		(property "Footprint" "Resistor_SMD:R_0201_0603Metric_Pad0.64x0.40mm_HandSolder"
+			(at 176.53 338.328 90)
+			(hide yes)
+			(show_name no)
+			(do_not_autoplace no)
+			(effects
+				(font
+					(size 1.27 1.27)
+				)
+			)
+		)
+		(property "Datasheet" ""
+			(at 176.53 336.55 0)
+			(hide yes)
+			(show_name no)
+			(do_not_autoplace no)
+			(effects
+				(font
+					(size 1.27 1.27)
+				)
+			)
+		)
+		(property "Description" "Resistor"
+			(at 176.53 336.55 0)
+			(hide yes)
+			(show_name no)
+			(do_not_autoplace no)
+			(effects
+				(font
+					(size 1.27 1.27)
+				)
+			)
+		)
+		(pin "2"
+		)
+		(pin "1"
+		)
+		(instances
+			(project "board"
+				(path "/27e6fb8b-ebcf-4ece-872b-7722c171602a"
+					(reference "R50")
+					(unit 1)
+				)

Commit message: Added power supply
Parts:
- added C11, C40: 22uF, Capacitor_SMD:C_1206_3216Metric_Pad1.33x1.80mm_HandSolder, symbol Device:C
- added C52, C53, C54, C55, C56, C57, C58, C59, C6, C60, C61, C62, C63, C64, C65, C66, C67, C68, C69, C70, C71, C72, C73, C74, C75, C76, C77, C78, C79, C80, C81, C82, C83, C84, C85, C86, C87, C88, C89, C90, C91: 100nF, Capacitor_SMD:C_0603_1608Metric, symbol Device:C
- added C8, C9: 10uF, Capacitor_SMD:C_1808_4520Metric_Pad1.72x2.30mm_HandSolder, symbol Device:C
- added C92: 0.1uF, Capacitor_SMD:C_1808_4520Metric_Pad1.72x2.30mm_HandSolder, symbol Device:C
- added L1: 2.2uH, leadedind:IND_1111-WE-TIS_WRE, symbol Device:L
- added R51: 33.2k, Resistor_THT:R_Axial_DIN0204_L3.6mm_D1.6mm_P5.08mm_Horizontal, symbol Device:R
- added R52, R53: 10k, Resistor_THT:R_Axial_DIN0204_L3.6mm_D1.6mm_P5.08mm_Horizontal, symbol Device:R
- added U22: TPS565201DDCT, psu:DDC0006A_N, symbol psu:TPS565201DDCT
- renumbered C6 to C48, C8 to C49, C9 to C50, C11 to C51
Connections:
- net GND: now also C11.2, C40.2, C52.2, C53.2, C54.2, C55.2, C56.2, C57.2, C58.2, C59.2, C6.2, C60.2, C61.2, C62.2, C63.2, C64.2, C65.2, C66.2, C67.2, C68.2, C69.2, C70.2, C71.2, C72.2, C73.2, C74.2, C75.2, C76.2, C77.2, C78.2, C79.2, C8.2, C80.2, C81.2, C82.2, C83.2, C84.2, C85.2, C86.2, C87.2, C88.2, C89.2, C9.2, C90.2, C91.2, R52.2, U22.1 (GND)
- net VCC: now also C11.1, C40.1, L1.2, R51.1
- net VCC5: now also C6.1, C8.1, C9.1, R53.1, U22.3 (VIN)
- new net: C92.1, L1.1, U22.2 (SW)
- new net: C92.2, U22.6 (VBST)
- new net: R51.2, R52.1, U22.4 (VFB)
- new net: R53.2, U22.5 (EN)
- new net vcc: C52.1, C53.1, C54.1, C55.1, C56.1, C57.1, C58.1, C59.1, C60.1, C61.1, C62.1, C63.1, C64.1, C65.1, C66.1, C67.1, C68.1, C69.1, C70.1, C71.1, C72.1, C73.1, C74.1, C75.1, C76.1, C77.1, C78.1, C79.1, C80.1, C81.1, C82.1, C83.1, C84.1, C85.1, C86.1, C87.1, C88.1, C89.1, C90.1, C91.1

Commit message: Re-organised power supply and added power connector
Parts:
- removed C47: 100nF, Capacitor_SMD:C_0603_1608Metric, symbol Device:C
- added J12: Conn_01x02_Socket, powerIn:CONN_SD-5566-002_02_MOL, symbol Connector:Conn_01x02_Socket
- C92: footprint Capacitor_SMD:C_1808_4520Metric_Pad1.72x2.30mm_HandSolder -> Capacitor_SMD:C_0603_1608Metric_Pad1.08x0.95mm_HandSolder
Connections:
- net vcc is gone; now on net VCC: C52.1, C53.1, C54.1, C55.1, C56.1, C57.1, C58.1, C59.1, C60.1, C61.1, C62.1, C63.1, C64.1, C65.1, C66.1, C67.1, C68.1, C69.1, C70.1, C71.1, C72.1, C73.1, C74.1, C75.1, C76.1, C77.1, C78.1, C79.1, C80.1, C81.1, C82.1, C83.1, C84.1, C85.1, C86.1, C87.1, C88.1, C89.1, C90.1, C91.1
- net GND: now also J12.1 (Pin_1)
- net VCC5: now also J12.2 (Pin_2)
Other:
- moved on the sheet: C33, C34

Commit message: Just before re-wiring the Mach to match the simulation
Parts:
- added D12, D13: LED, LED_SMD:LED_1206_3216Metric, symbol Device:LED
- added R54: 270, Resistor_SMD:R_0805_2012Metric_Pad1.20x1.40mm_HandSolder, symbol Device:R
- added R55: 412R, Resistor_SMD:R_0603_1608Metric, symbol Device:R
- added R56, R58, R59: 33R, Resistor_SMD:R_0201_0603Metric_Pad0.64x0.40mm_HandSolder, symbol Device:R
- added R57, R60, R61: 22R, Resistor_SMD:R_0201_0603Metric_Pad0.64x0.40mm_HandSolder, symbol Device:R
Connections:
- net EPROM_BUFFER_OE: now also R60.2
- net EPROM_CS: now also R58.2
- net EPROM_OE: now also R61.2
- net GND: now also D12.1 (K), D13.1 (K)
- net RAM_CS: now also R56.1
- net RAM_OE: now also R57.1
- net RW: now also R59.1
- net VCC: now also R54.2
- net VCC5: now also R55.2
- new net: D13.2 (A), R55.1
- new net: D12.2 (A), R54.1
Other:
- moved on the sheet: C1, C10, C11, C12, C13, C14, C15, C16, C17, C18, C19, C2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

Commit message: General save whilst getting eprom timing ok
Parts:
- removed R58: 33R, Resistor_SMD:R_0201_0603Metric_Pad0.64x0.40mm_HandSolder, symbol Device:R
- removed R60, R61: 22R, Resistor_SMD:R_0201_0603Metric_Pad0.64x0.40mm_HandSolder, symbol Device:R
